File: KiCad/SEGA_GamePad/SEGA_GamePad.kicad_pcb (KiCad board)
At the start: 2 copper layers, 32 x 53 mm, 36 parts, among them U1 AMS1117-3.3, U3 74HC14

Commit message: 13.03.2023 - 3D, KiCad, code
Connections:
- C11 pad 1: 5V -> 3.3V
- C12 pad 1: 5V -> 3.3V
- R10 pad 1: 5V -> 3.3V
- R11 pad 1: 5V -> 3.3V
- R13 pad 2: 5V -> 3.3V
- R15 pad 2: 5V -> 3.3V
- R16 pad 2: 5V -> 3.3V
- R9 pad 1: 5V -> 3.3V
- SEGA Gamepad v1.0 pad 5: 5V -> 3.3V
- U3 pad 14: 5V -> 3.3V
Routing:
- net 5V: track 102.5 -> 13.4 mm, vias 2 -> 1
- net 3.3V: track 192.4 -> 280.2 mm, vias 5 -> 6
