File: KiCad/SEGA_GamePad/SEGA_GamePad.sch (KiCad schematic (older format))
At the start: 36 parts, among them J1 Serial wire, J2 USB, J3 SEGA, U1 AMS1117-3.3, U2 STM32F103C8Tx, U3 74HC14, Y1 8MHz

Commit message: 13.03.2023 - 3D, KiCad, code
Connections:
- net 3.3V: now also C11.1, C12.1, U3.14 (VCC)
- net 5V: no longer C11.1, C12.1, U3.14 (VCC)
Changed lines of the file:
@@
 $EndComp
 Text GLabel 1050 4200 1    50   Input ~ 0
-5V
+3.3V
 $Comp
 L power:GND #PWR011
